Commit message: Fixed puma260 urdf, fixed deployer, fixed stupid issue, velocity command for puma260 doesn't work, wrong puma260 urdf mesh origins

File: robots/puma260/puma260_description/robots/puma260.urdf (robot description, URDF)
Before this commit: robot puma260, 7 links, 6 joints
Links:
- link arm: geometry visual mesh filename=package://puma260_description/meshes/arm.stl
- link base_link: geometry visual mesh filename=package://puma260_description/meshes/base_link.stl
- link end_effector: geometry visual mesh filename=package://puma260_description/meshes/end_effector.stl
- link forearm: geometry visual mesh filename=package://puma260_description/meshes/forearm.stl
- link link_dummy_1: geometry visual mesh filename=package://puma260_description/meshes/link_dummy_1.stl
- link link_dummy_2: geometry visual mesh filename=package://puma260_description/meshes/link_dummy_2.stl
- link torso: geometry visual mesh filename=package://puma260_description/meshes/torso.stl
Joints:
- joint joint_1: origin xyz=0.0 0.0 0.3302 -> xyz=0.0 0.0 0.0 rpy=0.0 0.0 0.0
- joint joint_2: origin xyz=0.0 +0.067 0.0 rpy=1.5708 0 0 -> xyz=0.0 0.0 0.3302 rpy=-1.5708 0.38 0.0 
- joint joint_3: origin xyz=0.1362 0.0 -0.0597 rpy=0 0 0 -> xyz=0.203202 0.0 0.0 rpy=0.0 0.0 0.0
- joint joint_4: origin xyz=0.2032 0.0 0.0 rpy=0 1.5708 0 -> xyz=0.0 0.0 -0.12623 rpy=1.57 0.0 3.42
- joint joint_5: origin xyz=0.0 0.0 0.0 rpy=0 1.5708 0 -> xyz=0.0 0.0 0.2032 rpy=-1.5708 0.0 1.57059
- joint joint_6: origin xyz=-0.019 0.0 0.0 rpy=0 -1.5708 0 -> xyz=0.0 0.0 0.0 rpy=1.57 0.0 -1.57
