Commit message: fixed robot names, wam nodes and added newrun.sh which should work just fine

File: robots/wam7dof/wam7dof_description/robots/wam7dof.urdf (robot description, URDF)
Before this commit: robot wam, 10 links, 9 joints
Links:
- removed link wam/base_link
- removed link wam/forearm_link
- removed link wam/shoulder_pitch_link
- removed link wam/shoulder_yaw_link
- removed link wam/upper_arm_link
- removed link wam/wrist_palm_link
- removed link wam/wrist_palm_stump_link
- removed link wam/wrist_pitch_link
- removed link wam/wrist_yaw_link
- added link base_link, mass 1; collision mesh filename=package://wam7dof_description/models/sw_meshes/base_link_co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; visual mesh filename=package://wam7dof_description/models/sw_meshes/base_link_fi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
- added link forearm_link, mass 0.50016804; collision mesh filename=package://wam7dof_description/models/sw_meshes/elbow_link_c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; collision mesh filename=package://wam7dof_description/models/sw_meshes/forearm_link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
- added link shoulder_pitch_link, mass 3.87493756; collision mesh filename=package://wam7dof_description/models/sw_meshes/shoulder_pit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; visual mesh filename=package://wam7dof_description/models/sw_meshes/shoulder_pit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
- added link shoulder_yaw_link, mass 5.0; collision mesh filename=package://wam7dof_description/models/sw_meshes/shoulder_lin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; visual mesh filename=package://wam7dof_description/models/sw_meshes/shoulder_lin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
- added link upper_arm_link, mass 2.20228141; collision mesh filename=package://wam7dof_description/models/sw_meshes/upper_arm_li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; visual mesh filename=package://wam7dof_description/models/sw_meshes/upper_arm_li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
- added link wrist_palm_link, mass 0.08286134; collision mesh filename=package://wam7dof_description/models/sw_meshes/wrist_palm_l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; visual mesh filename=package://wam7dof_description/models/sw_meshes/wrist_palm_l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
- added link wrist_palm_stump_link, mass 0.000001
- added link wrist_pitch_link, mass 0.51797364; collision mesh filename=package://wam7dof_description/models/sw_meshes/wrist_pitch_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; visual mesh filename=package://wam7dof_description/models/sw_meshes/wrist_pitch_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
- added link wrist_yaw_link, mass 1.05376019; collision mesh filename=package://wam7dof_description/models/sw_meshes/wrist_yaw_li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; visual mesh filename=package://wam7dof_description/models/sw_meshes/wrist_yaw_li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
Joints:
- removed joint wam/base_yaw_joint
- removed joint wam/elbow_pitch_joint
- removed joint wam/palm_yaw_joint
- removed joint wam/shoulder_pitch_joint
- removed joint wam/shoulder_yaw_joint
- removed joint wam/wam_fixed_joint
- removed joint wam/wrist_palm_stump_joint
- removed joint wam/wrist_pitch_joint
- removed joint wam/wrist_yaw_joint
- added joint base_yaw_joint: type revolute, parent base_link, child shoulder_yaw_link, origin xyz=0 0 0.346 rpy=0 0 0, axis 0 0 1, limit lower=-2.6 upper=2.6 effort=60 velocity=2.0
- added joint elbow_pitch_joint: type revolute, parent upper_arm_link, child forearm_link, origin xyz=0.045 0 0.55 rpy=-1.57079632679 0 0, axis 0 0 1, limit lower=-0.9 upper=3.14159265359 effort=30 velocity=2.00
- added joint palm_yaw_joint: type revolute, parent wrist_pitch_link, child wrist_palm_link, origin xyz=0 0 0 rpy=1.57079632679 0 0, axis 0 0 1, limit lower=-3.0 upper=3.0 effort=10 velocity=2.00
- added joint shoulder_pitch_joint: type revolute, parent shoulder_yaw_link, child shoulder_pitch_link, origin xyz=0 0 0 rpy=-1.57079632679 0 0, axis 0 0 1, limit lower=-1.985 upper=1.985 effort=60 velocity=2.0
- added joint shoulder_yaw_joint: type revolute, parent shoulder_pitch_link, child upper_arm_link, origin xyz=0 0 0 rpy=1.57079632679 0 0, axis 0 0 1, limit lower=-2.8 upper=2.8 effort=45 velocity=2.0
- added joint wam_fixed_joint: type fixed, parent world, child base_link, origin xyz=0.0 0.0 1.0 rpy=0 0 0
- added joint wrist_palm_stump_joint: type fixed, parent wrist_palm_link, child wrist_palm_stump_link, origin xyz=0 0 0.06 rpy=0 0 0
- added joint wrist_pitch_joint: type revolute, parent wrist_yaw_link, child wrist_pitch_link, origin xyz=0 0 0 rpy=-1.57079632679 0 0, axis 0 0 1, limit lower=-1.5707 upper=1.5707 effort=10 velocity=2.00
- added joint wrist_yaw_joint: type revolute, parent forearm_link, child wrist_yaw_link, origin xyz=-0.045 -0.3 0 rpy=1.57079632679 0 0, axis 0 0 1, limit lower=-4.55 upper=1.25 effort=10 velocity=2.0

Commit message: modified youbot name and some capitalization issue

File: robots/wam7dof/wam7dof_description/robots/wam7dof.urdf (robot description, URDF)
Before this commit: robot wam, 10 links, 9 joints
Joints:
- removed joint base_yaw_joint
- removed joint elbow_pitch_joint
- removed joint palm_yaw_joint
- removed joint shoulder_pitch_joint
- removed joint shoulder_yaw_joint
- removed joint wam_fixed_joint
- removed joint wrist_palm_stump_joint
- removed joint wrist_pitch_joint
- removed joint wrist_yaw_joint
- added joint joint_0: type fixed, parent world, child base_link, origin xyz=0.0 0.0 1.0 rpy=0 0 0
- added joint joint_1: type revolute, parent base_link, child shoulder_yaw_link, origin xyz=0 0 0.346 rpy=0 0 0, axis 0 0 1, limit lower=-2.6 upper=2.6 effort=60 velocity=2.0
- added joint joint_2: type revolute, parent shoulder_yaw_link, child shoulder_pitch_link, origin xyz=0 0 0 rpy=-1.57079632679 0 0, axis 0 0 1, limit lower=-1.985 upper=1.985 effort=60 velocity=2.0
- added joint joint_3: type revolute, parent shoulder_pitch_link, child upper_arm_link, origin xyz=0 0 0 rpy=1.57079632679 0 0, axis 0 0 1, limit lower=-2.8 upper=2.8 effort=45 velocity=2.0
- added joint joint_4: type revolute, parent upper_arm_link, child forearm_link, origin xyz=0.045 0 0.55 rpy=-1.57079632679 0 0, axis 0 0 1, limit lower=-0.9 upper=3.14159265359 effort=30 velocity=2.00
- added joint joint_5: type revolute, parent forearm_link, child wrist_yaw_link, origin xyz=-0.045 -0.3 0 rpy=1.57079632679 0 0, axis 0 0 1, limit lower=-4.55 upper=1.25 effort=10 velocity=2.0
- added joint joint_6: type revolute, parent wrist_yaw_link, child wrist_pitch_link, origin xyz=0 0 0 rpy=-1.57079632679 0 0, axis 0 0 1, limit lower=-1.5707 upper=1.5707 effort=10 velocity=2.00
- added joint joint_7: type revolute, parent wrist_pitch_link, child wrist_palm_link, origin xyz=0 0 0 rpy=1.57079632679 0 0, axis 0 0 1, limit lower=-3.0 upper=3.0 effort=10 velocity=2.00
- added joint joint_8: type fixed, parent wrist_palm_link, child wrist_palm_stump_link, origin xyz=0 0 0.06 rpy=0 0 0
